File: pcb/requirements.kicad_sch (KiCad schematic)
At the start: 0 parts

Commit message: Standardized parts; fixed title box
Other:
- title: Relay Module -> Servo Module
Changed lines of the file:
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@@
 	(paper "A4")
 	(title_block
-		(title "Relay Module")
+		(title "Servo Module")
 		(date "<<release-date>>")
 		(rev "<<tag>>")
