File: pcb/requirements.kicad_sch (KiCad schematic)
At the start: 10 parts

Commit message: Converted to Kicad10
Parts:
- LOGO1, LOGO2, LOGO3, LOGO5, LOGO6: value ~ -> (none)

Commit message: Added decoupling per servo
Updated silkscreen instructions
Refitted for guardrail
Updated renders
Parts:
- LOGO5: footprint CRGM Logos:Roxy 5mm -> CRGM Logos:Roxy 4mm
Changed lines of the file:
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@@
 		)
 	)
-	(text_box "BASIC\n\n* STM32C0 Processor\n* 48MHz Crystal\n* Adafruit Seesaw Protocol\n* Four Servo Ports\n* Power In/Out Ports\n* Optional Pull Ups for I2C\n* I2C Address Selection (2-bits)\n* Servo Power Connector\n* Servo Power Indicator\n* Servo Status Indicators\n"
+	(text_box "BASIC\n\n* STM32C0 Processor\n* 48MHz Crystal\n* Adafruit Seesaw Protocol\n* Four Servo Ports\n* Power In/Out Ports\n* Optional Pull Ups for I2C\n* I2C Address Selection (2-bits)\n"
 		(exclude_from_sim yes)
 		(at 19.05 32.385 0)
@@
 		)
 	)
-	(text_box "Servo Specifications\n\n* 5V, 90g\n* 0-180 Degrees\n* Standard PWM\n"
+	(text_box "Servo Specifications\n\n* 5V, 90g\n* 0-180 Degrees\n* Standard PWM\n* Servo Power Connector\n* Servo Power Indicator\n* Servo Status Indicators\n* Bulk and Decoupling Caps"
 		(exclude_from_sim yes)
 		(at 90.17 32.385 0)
@@
 		(property "Mouser" ""
 			(at 158.75 171.45 0)
+			(hide yes)
+			(show_name no)
+			(do_not_autoplace no)
+			(effects
+				(font
+					(size 1.27 1.27)
+				)
+			)
+		)
+		(property "WVDC" ""
+			(at 158.75 171.45 90)
 			(hide yes)
 			(show_name no)
@@
 			)
 		)
+		(property "WVDC" ""
+			(at 36.83 186.69 0)
+			(hide yes)
+			(show_name no)
+			(do_not_autoplace no)
+			(effects
+				(font
+					(size 1.27 1.27)
+				)
+			)
+		)
 		(instances
 			(project "servo-module"
@@
 		(property "MPN" ""
 			(at 158.75 181.61 0)
+			(show_name no)
+			(do_not_autoplace no)
+			(effects
+				(font
+					(size 1.27 1.27)
+				)
+			)
+		)
+		(property "WVDC" ""
+			(at 158.75 181.61 90)
+			(hide yes)
 			(show_name no)
 			(do_not_autoplace no)
@@
 			)
 		)
+		(property "WVDC" ""
+			(at 60.96 186.69 0)
+			(hide yes)
+			(show_name no)
+			(do_not_autoplace no)
+			(effects
+				(font
+					(size 1.27 1.27)
+				)
+			)
+		)
 		(instances
 			(project "servo-module"
@@
 			)
 		)
+		(property "WVDC" ""
+			(at 85.09 186.69 0)
+			(hide yes)
+			(show_name no)
+			(do_not_autoplace no)
+			(effects
+				(font
+					(size 1.27 1.27)
+				)
+			)
+		)
 		(instances
 			(project "servo-module"
@@
 			)
 		)
+		(property "WVDC" ""
+			(at 158.75 176.53 90)
+			(hide yes)
+			(show_name no)
+			(do_not_autoplace no)
+			(effects
+				(font
+					(size 1.27 1.27)
+				)
+			)
+		)
 		(pin "1"
 		)
@@
 		)
 		(property "Description" ""
+			(at 48.26 186.69 0)
+			(hide yes)
+			(show_name no)
+			(do_not_autoplace no)
+			(effects
+				(font
+					(size 1.27 1.27)
+				)
+			)
+		)
+		(property "WVDC" ""
 			(at 48.26 186.69 0)
 			(hide yes)
@@
 			)
 		)
+		(property "WVDC" ""
+			(at 25.4 186.69 0)
+			(hide yes)
+			(show_name no)
+			(do_not_autoplace no)
+			(effects
+				(font
+					(size 1.27 1.27)
+				)
+			)
+		)
 		(instances
 			(project "servo-module"
@@
 			)
 		)
-		(property "Footprint" "CRGM Logos:Roxy 5mm"
+		(property "Footprint" "CRGM Logos:Roxy 4mm"
 			(at 73.66 194.818 0)
 			(hide yes)
@@
 		)
 		(property "Mouser" ""
+			(at 73.66 186.69 0)
+			(hide yes)
+			(show_name no)
+			(do_not_autoplace no)
+			(effects
+				(font
+					(size 1.27 1.27)
+				)
+			)
+		)
+		(property "WVDC" ""
+			(at 73.66 186.69 0)
+			(hide yes)
+			(show_name no)
+			(do_not_autoplace no)
+			(effects
+				(font
+					(size 1.27 1.27)
+				)
+			)
+		)
+		(property "MN" ""
+			(at 73.66 186.69 0)
+			(hide yes)
+			(show_name no)
+			(do_not_autoplace no)
+			(effects
+				(font
+					(size 1.27 1.27)
+				)
+			)
+		)
+		(property "MPN" ""
 			(at 73.66 186.69 0)
 			(hide yes)
@@
 			(show_name no)
 			(do_not_autoplace no)
+			(effects
+				(font
+					(size 1.27 1.27)
+				)
+			)
+		)
+		(property "WVDC" ""
+			(at 158.75 186.69 90)
+			(hide yes)
+			(show_name no)
+			(do_not_autoplace no)
