File: pcb/mcu.kicad_sch (KiCad schematic)
At the start: 28 parts, among them J1 SWD Header, SW1 SKRPABE010, U1 STM32C031G6Ux, Y1 ECS-480-10-37B2-RWN-TR

Commit message: removed space
Parts:
- R1, R2: MN FOJAN -> FOJAN
Changed lines of the file:
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@@
 			)
 		)
-		(property "MN" "FOJAN "
+		(property "MN" "FOJAN"
 			(at 46.99 66.04 0)
 			(effects
@@
 			)
 		)
-		(property "MN" "FOJAN "
+		(property "MN" "FOJAN"
 			(at 53.34 66.04 0)
 			(effects

Commit message: Updated MN and MPN
Parts:
- J1: MN (none) -> DEALON; MPN (none) -> DZ127S-22-10-55
- U1: MN (none) -> STMicroelectronics; MPN (none) -> STM32C031G6U6TR
Changed lines of the file:
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@@
+			)
+		)
+		(property "MN" "STMicroelectronics"
+			(at 107.95 66.04 0)
+			(effects
+				(font
+					(size 1.27 1.27)
+				)
+				(hide yes)
+			)
+		)
+		(property "MPN" "STM32C031G6U6TR"
+			(at 107.95 66.04 0)
+			(effects
+				(font
+					(size 1.27 1.27)
+				)
+				(hide yes)
 			)
 		)
@@
 			(at 231.14 48.26 0)
 			(effects
+				(font
+					(size 1.27 1.27)
+				)
+				(hide yes)
+			)
+		)
+		(property "MN" "DEALON"
+			(at 231.14 48.26 0)
+			(effects
+				(font
+					(size 1.27 1.27)
+				)
+				(hide yes)
+			)
+		)
+		(property "MPN" "DZ127S-22-10-55"
+			(at 231.14 48.26 0)
+			(effects
