File: pcb/mcu.kicad_sch (KiCad schematic)
At the start: 28 parts, among them J1 SWD Header, SW1 SKRPABE010, U1 STM32C031G6Ux, Y1 ECS-480-10-37B2-RWN-TR

Commit message: Converted to Kicad10
Parts:
- JP1, JP2, JP3, JP4, TP1, TP10, TP2, TP3, TP9: value ~ -> (none)

Commit message: Added decoupling per servo
Updated silkscreen instructions
Refitted for guardrail
Updated renders
Other:
- moved on the sheet: C1, C2, C5, D1, D2, D3, D4, JP1, JP2, JP3, JP4, R1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

Commit message: Upgraded to STM32C051G8
Parts:
- U1: value STM32C031G6Ux -> STM32C051G8Ux; symbol CRG Makes:STM32C031G6Ux -> CRG Makes:STM32C051G8Ux; Digikey 497-STM32C031G6U6-ND -> 497-STM32C051G8U6-ND; LCSC C7324966 -> C44847692; MN STMicroelectronics -> (none); MPN STM32C031G6U6TR -> (none); Mouser 511-STM32C031G6U6 -> 511-STM32C051G8U6
Changed lines of the file:
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@@
 	)
 	(symbol
-		(lib_id "CRG Makes:STM32C031G6Ux")
+		(lib_id "CRG Makes:STM32C051G8Ux")
 		(at 109.22 69.85 0)
 		(unit 1)
@@
 			)
 		)
-		(property "Value" "STM32C031G6Ux"
+		(property "Value" "STM32C051G8Ux"
 			(at 113.03 45.72 0)
 			(show_name no)
@@
 			)
 		)
-		(property "Datasheet" "https://www.st.com/resource/en/datasheet/stm32c031g6.pdf"
+		(property "Datasheet" "https://www.st.com/resource/en/datasheet/stm32c051g8.pdf"
 			(at 109.22 113.03 0)
 			(hide yes)
@@
 			)
 		)
-		(property "Description" "STMicroelectronics Arm Cortex-M0+ MCU, 32KB flash, 12KB RAM, 48 MHz, 2.0-3.6V, 26 GPIO, UFQFPN28"
+		(property "Description" "-40℃~+85℃ 12KB 26 2V~3.6V 32 Bit 48MHz 64KB ARM Cortex-M0+ Built-in FLASH UFQFPN-28(4x4)"
 			(at 109.22 108.204 0)
 			(hide yes)
@@
 			)
 		)
-		(property "Digikey" "497-STM32C031G6U6-ND"
+		(property "Digikey" "497-STM32C051G8U6-ND"
 			(at 109.22 115.57 0)
 			(hide yes)
@@
 			)
 		)
-		(property "Mouser" "511-STM32C031G6U6"
+		(property "Mouser" "511-STM32C051G8U6"
 			(at 109.22 118.11 0)
 			(hide yes)
@@
 			)
 		)
-		(property "LCSC" "C7324966"
+		(property "LCSC" "C44847692"
 			(at 109.22 120.65 0)
 			(hide yes)
 			(show_name no)
-			(do_not_autoplace no)
-			(effects
-				(font
-					(size 1.27 1.27)
-				)
-			)
-		)
-		(property "MN" "STMicroelectronics"
-			(at 109.22 69.85 0)
-			(hide yes)
-			(show_name no)
-			(do_not_autoplace no)
-			(effects
-				(font
-					(size 1.27 1.27)
-				)
-			)
-		)
-		(property "MPN" "STM32C031G6U6TR"
-			(at 109.22 69.85 0)
-			(hide yes)
-			(show_name no)
-			(do_not_autoplace no)
-			(effects
-				(font
-					(size 1.27 1.27)
-				)
-			)
-		)
-		(property "WVDC" ""
-			(at 109.22 69.85 0)
-			(hide yes)
-			(show_name no)

Commit message: Updated symbols
Parts:
- JP1, JP2: value (none) -> SolderJumper_2_Open
- JP3, JP4: value (none) -> SolderJumper_2_Open; symbol Jumper:SolderJumper_2_Open -> CRGM Connector:SolderJumper_2_Open
Connections:
- net SCL: no longer JP1.1 (A)
- net SDA: no longer JP2.1 (A)
- net at JP2.2 (B): no longer R2.1
- net at JP1.2 (B): no longer R1.1
Other:
- moved on the sheet: JP3, JP4
